File: pcb/nixie_clock/nixie_clock.brd (EAGLE design)
At the start: 140 x 70 mm, 38 parts, among them Q1 IRLR3110ZPBF, T1 DA2032-AL, U1 ESP32, U2 CP2102N, U3 LT3757

Commit message: sch and pcb outline
Parts:
- added C12: 0.22F, Passive Components > Capacitors > Supercapacitors \ Ultracapacitors:DSK-614/621
- added C13, C14, C18, C19: 1u, Passive Components > Capacitors > Multilayer Ceramic Capacitors MLCC:0603_WAVE
- added C15: 22n, Passive Components > Capacitors > Multilayer Ceramic Capacitors MLCC:0603_WAVE
- added C16, C17, C20, C23, C26, C27, C28, C29, C30, C31, C40: 100n, Passive Components > Capacitors > Multilayer Ceramic Capacitors MLCC:0603_WAVE
- added C21: 4u7, Passive Components > Capacitors > Multilayer Ceramic Capacitors MLCC:0603_WAVE
- added C22: 100p, Passive Components > Capacitors > Multilayer Ceramic Capacitors MLCC:0603_WAVE
- added C24, C25: 15p, Passive Components > Capacitors > Multilayer Ceramic Capacitors MLCC:0603_WAVE
- added C32: 10n, Passive Components > Capacitors > Multilayer Ceramic Capacitors MLCC:0603_WAVE
- added C33: 3n, Passive Components > Capacitors > Multilayer Ceramic Capacitors MLCC:0603_WAVE
- added C34, C35: 270p, Passive Components > Capacitors > Multilayer Ceramic Capacitors MLCC:0603_WAVE
- added C36, C37: 10p, Passive Components > Capacitors > Multilayer Ceramic Capacitors MLCC:0603_WAVE
- added C38: 5p6, Passive Components > Capacitors > Multilayer Ceramic Capacitors MLCC:0603_WAVE
- added C39: 2p4, Passive Components > Capacitors > Multilayer Ceramic Capacitors MLCC:0603_WAVE
- added D6: B0530W, Semiconductors > Discrete Semiconductors > Diodes & Rectifiers > Schottky Diodes & Rectifiers:SOD-123
- added D7, D8: LED0603, Opto-electronics > LED Emitters:CHIPLED_0603
- added F1: (no value), Circuit Protection > Resettable Fuses - PPTC:0805
- added J1: USB-C, Connectors > USB:USB-C
- added L1: 10u, Passive Components > Inductors, Chokes & Coils:_1210
- added L2: 2n7, Passive Components > Inductors, Chokes & Coils:_0603
- added NL1, NL2: NEON6X16, vacuum_tubes:NL-6X16
- added Q2, Q3, Q4, Q5, Q6, Q7: BC817-25, Semiconductors > Discrete Semiconductors > Transistors > Bipolar Transistors - BJT:SOT-23-3
- added R13: 94k, Passive Components > Resistors > Chip Resistors:0603_WAVE
- added R14, R16, R25, R33, R34, R35: 10k, Passive Components > Resistors > Chip Resistors:0603_WAVE
- added R15: 85k, Passive Components > Resistors > Chip Resistors:0603_WAVE
- added R17, R18: 100k, Passive Components > Resistors > Chip Resistors:_1206
- added R23, R24, R28, R29: 11k5, Passive Components > Resistors > Chip Resistors:0603_WAVE
- added R26: 47k5, Passive Components > Resistors > Chip Resistors:0603_WAVE
- added R27: 22k1, Passive Components > Resistors > Chip Resistors:0603_WAVE
- added R30, R31, R38: 1k, Passive Components > Resistors > Chip Resistors:0603_WAVE
- added R32: 20k, Passive Components > Resistors > Chip Resistors:0603_WAVE
- added R36, R37: 4k7, Passive Components > Resistors > Chip Resistors:0603_WAVE
- added SW1, SW2: (no value), Eletromechanical > Switches > Tactile Switches:PUSH_BUTTON
- added U$1: MIC2619, Power > Switching Controllers:SOT-23-6N
- added U4: DS3231, Semiconductors > Integrated Circuits - ICs > Clock & Timer ICs > Real Time Clock:SOIC-16
- added U5, U6: HV5522, Power > Power Switch:QFP64
- added U7: MCP1700T-3302TT, Power > LDO Voltage Regulators:SOT-23
- added U8: W25Q40BVSS, Semiconductors > Integrated Circuits - ICs > Memory ICs > Flash:SO08-SS
- added X1: 32.768kHz, Passive Components > Frequency Control & Timing Devices > Crystals:2-SMD-3215
- added X2: 26MHz, Passive Components > Frequency Control & Timing Devices > Crystals:4-SMD-3225
- R10, R11, R12, R9: value (none) -> 15k
- moved R10 184.8 mm to (-40.6, 69.8)
- moved R7 183.1 mm to (-53.3, 74.9)
- moved R9 179.0 mm to (-34.3, 69.8)
- moved R4 178.6 mm to (-49.5, 74.9)
- moved C11 170.0 mm to (-34.3, 74.9)
- moved C10 165.6 mm to (-30.5, 74.9)
- moved D4 163.1 mm to (-72.4, 69.8), turned to 0 degrees
- moved C9 161.3 mm to (-26.7, 74.9)
- moved R5 161.0 mm to (-40.6, 62.2)
- moved C8 157.1 mm to (-22.9, 74.9)
- moved C7 152.9 mm to (-19.1, 74.9)
- moved R8 143.4 mm to (-47.0, 62.2)
- moved R3 137.0 mm to (-45.7, 74.9)
- moved R6 136.5 mm to (-30.5, 63.5)
- moved D5 135.6 mm to (-15.2, 76.2), turned to 0 degrees
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Connections:
- new net !DSP_BL: U1.14
- new net !DSP_LE: U1.21
- new net 12V: C14.P$1, C15.P$1, C16.P$1, C17.P$1, D6.C, R13.P$2, R15.P$2, U5.27, U5.30, U6.27, U6.30
- new net 3.3V: C19.P$1, C20.P$1, C21.P$1, C22.P$1, C23.P$1, C26.P$1, C27.P$1, C28.P$1, C30.P$1, C31.P$1, C40.P$1, R25.P$2, R28.P$2, R29.P$2, R35.P$2, R36.P$2, R37.P$2, R38.P$2, U1.1, U1.19, U1.3, U1.37, U1.4, U1.43, U1.46, U2.5, U2.6, U2.7, U4.2, U7.2, U8.8
- new net CHIP_PU: Q3.P$3, R28.P$1, SW1.LB, SW1.RB, U1.9
- new net DSP_BL_CLK: D2.4, U1.35
- new net DSP_BL_SDI: D2.3, U1.36
- new net DSP_CLK: U1.17
- new net DSP_SDI: U1.20
- new net DTR: Q2.P$2, R34.P$2, U2.23
- new net FLASH_SCK: U1.31, U8.6
- new net FLASH_SCS: U1.30, U8.1
- new net FLASH_SDI: U1.33, U8.5
- new net FLASH_SDO: U1.32, U8.2
- new net FLASH_SHD: U1.28, U8.7
- new net FLASH_SWP: U1.29, U8.3
- new net FLASH_VDD: C29.P$1, U1.26
- new net GPIO0-BOOT: Q2.P$3, R29.P$1, SW2.LB, SW2.RB, U1.23
- new net HFXTAL_N: C36.P$1, U1.44, X2.1
- new net HFXTAL_P: C37.P$1, U1.45, X2.3
- new net LED: D7.A, U1.34
- new net LFXTAL_N: C25.P$1, U1.13, X1.2
- new net LFXTAL_P: C24.P$1, U1.12, X1.1
- new net N$16: D6.A, L1.2, U$1.1
- new net N$17: R13.P$1, R14.P$2, U$1.5
- new net N$18: C15.P$2, R15.P$1, R16.P$2, U$1.3
- new net N$19: NL1.2, R17.1
- new net N$20: NL2.2, R18.1
- new net N$23: U5.23, U6.32
- new net N$72: D3.1, D4.3
- new net N$73: D3.6, D4.4
- new net N$74: F1.2, J1.A4/B9, J1.B4/A9
- new net N$75: J1.B5, R23.P$2
- new net N$76: D4.6, D5.4
- new net N$77: D4.1, D5.3
- new net N$78: J1.A5, R24.P$2
- new net N$79: R25.P$1, U2.9
- new net N$80: D8.C, R30.P$2
- new net N$81: D2.6, D3.4
- new net N$82: D2.1, D3.3
- new net N$83: R26.P$2, R27.P$1, U2.8
- new net N$84: D7.C, R31.P$2
- new net N$85: C33.P$1, R32.P$2, U1.47
- new net N$86: C34.P$1, U1.8
- new net N$87: C32.P$1, C33.P$2, R32.P$1, U1.48
- new net N$88: C35.P$1, U1.5
- new net N$89: C34.P$2, U1.7
- new net N$90: C35.P$2, U1.6
- new net N$91: C38.P$1, L2.2, U1.2
- new net N$92: Q2.P$1, R33.P$1
- new net N$93: Q3.P$1, R34.P$1
- new net N$94: C38.P$2, C39.P$1, E1.ANT
- new net N$95: C12.1, U4.14
- new net N$96: R35.P$1, U4.4
- new net NT1-0: NT1.0, U5.1
- new net NT1-1: NT1.1, U5.2
- new net NT1-2: NT1.2, U5.3
- new net NT1-3: NT1.3, U5.4
- new net NT1-4: NT1.4, U5.5
- new net NT1-5: NT1.5, U5.6
- new net NT1-6: NT1.6, U5.7
- new net NT1-7: NT1.7, U5.8
- new net NT1-8: NT1.8, U5.9
- new net NT1-9: NT1.9, U5.10
- new net NT2-0: NT2.0, U5.35
- new net NT2-1: NT2.1, U5.36
- new net NT2-2: NT2.2, U5.37
- new net NT2-3: NT2.3, U5.38
- new net NT2-4: NT2.4, U5.39
- new net NT2-5: NT2.5, U5.40
- new net NT2-6: NT2.6, U5.41
- new net NT2-7: NT2.7, U5.42
- new net NT2-8: NT2.8, U5.43
- new net NT2-9: NT2.9, U5.44
- new net RTC_INT: R38.P$1, U1.24, U4.3
- new net RTS: Q3.P$2, R33.P$2, U2.19
- new net SCL: R37.P$1, U1.39, U4.16
- new net SDA: R36.P$1, U1.42, U4.15
- new net U0RXD: U1.40, U2.21
- new net U0TXD: U1.41, U2.20
- new net USB_DM: J1.A7, J1.B7, U2.4
- new net USB_DP: J1.A6, J1.B6, U2.3
- net !HVEN: now also U1.15
- net 5V: now also C13.P$1, C18.P$1, D2.5, D3.5, D4.5, D5.5, D8.A, F1.1, L1.1, R27.P$2, U$1.4, U$1.6, U7.3
- net GND: now also C12.2, C13.P$2, C14.P$2, C16.P$2, C17.P$2, C18.P$2, C19.P$2, C20.P$2, C21.P$2, C22.P$2, C23.P$2, C24.P$2, C25.P$2, C26.P$2, C27.P$2, C28.P$2, C29.P$2, C30.P$2, C31.P$2, C32.P$2, C36.P$2, C37.P$2, C39.P$2, C40.P$2, D2.2, D3.2, D4.2, D5.2, E1.GND, J1.A1/B12, J1.B1/A12, J1.SHIELD0, J1.SHIELD1, J1.SHIELD2, J1.SHIELD3, L2.1, R14.P$1, R16.P$1, R23.P$1, R24.P$1, R26.P$1, R30.P$1, R31.P$1, SW1.LT, SW1.RT, SW2.LT, SW2.RT, U$1.2, U1.EP, U2.2, U2.PAD, U4.10, U4.11, U4.12, U4.13, U4.5, U4.6, U4.7, U4.8, U4.9, U5.29, U6.29, U7.1, U8.4, X2.2, X2.4
- net VOUT: now also R17.2, R18.2
Routing:
- net NT2-9: track 0.00 -> 50.2 mm
- net NT2-8: track 0.00 -> 43.3 mm
- net NT2-7: track 0.00 -> 37.1 mm
- net NT2-6: track 0.00 -> 31.8 mm
- net NT2-5: track 0.00 -> 26.6 mm
- net NT2-4: track 0.00 -> 21.9 mm
- net NT2-0: track 0.00 -> 19.8 mm
- net NT2-3: track 0.00 -> 17.7 mm
- net NT2-2: track 0.00 -> 13.5 mm
- net NT2-1: track 0.00 -> 9.90 mm
Other:
- board size 140 x 70 mm -> 130 x 50 mm

Commit message: rough pcb done
Parts:
- removed U$1: MIC2619, Power > Switching Controllers:SOT-23-6N
- added C41, C42, C43, C44: (no value), Passive Components > Capacitors > Multilayer Ceramic Capacitors MLCC:0603_WAVE
- added C45: 47u, Passive Components > Capacitors > Multilayer Ceramic Capacitors MLCC:_1210
- added D9: BAT54S, Semiconductors > Discrete Semiconductors > Diodes & Rectifiers > Schottky Diodes & Rectifiers:SOT-23-3
- added J2, J3: 8, Connectors > Header:1X8_2.54
- added J4, J5: 4, Connectors > Header:1X4_2.54
- added LOGO1, LOGO8: DESIGNEDINPT, Utility > Silkscreen:DESIGNEDINPT
- added LOGO2: RAFAEL_SILVA10CIRCLE, Utility > Silkscreen:RAFAEL_SILVA_10MM_CIRCLE
- added LOGO3, LOGO9: OSHW-LOGOL, Utility > Silkscreen:OSHW-LOGO-L
- added LOGO4, LOGO6: HV_WARNING, Silkscreen:HV_WARNING
- added LOGO5: RADIO-10MM, Silkscreen:RADIO_10MM
- added LOGO7: RAFAEL_SILVA10MM, Utility > Silkscreen:RAFAEL_SILVA_10MM
- added R19, R21, R22, R39, R40, R41, R42: 1k, Passive Components > Resistors > Chip Resistors:0603_WAVE
- added R20: 94k, Passive Components > Resistors > Chip Resistors:0603_WAVE
- added R43: 100, Passive Components > Resistors > Chip Resistors:0603_WAVE
- added R44: 10k, Passive Components > Resistors > Chip Resistors:0603_WAVE
- added U10, U11: 74LVC1G17, Semiconductors > Integrated Circuits - ICs > Logic ICs > Logic Gates:SC70-5
- added U9: MIC2619, Power > Switching Controllers:SOT-23-6N
- C33: value 3n -> 3n3
- E1: value ANTENNATRACE-15.2MM -> ANTENNATRACE; device Passive Components > Antennas:TRACE_ANTENNA_2.4GHZ_15.2MM -> Passive Components > Antennas:TRACE_ANTENNA_2.4GHZ_25.7MM
- R6: value 10k -> 100k
- R7: value 75k -> 10k
- SW1, SW2: device Eletromechanical > Switches > Tactile Switches:PUSH_BUTTON -> Eletromechanical > Switches > Tactile Switches:3X4X2
- U7: value MCP1700T-3302TT -> MIC39100; device Power > LDO Voltage Regulators:SOT-23 -> Power > LDO Voltage Regulators:SOT230P700X180-4N
- moved D6 303.4 mm to (116.2, 57.1), turned to 180 degrees
- moved C15 298.5 mm to (114.5, 60.0)
- moved R16 232.0 mm to (116.1, 63.1), turned to 270 degrees
- moved R14 230.3 mm to (117.7, 63.1), turned to 270 degrees
- moved R15 229.1 mm to (116.1, 60.0), turned to 270 degrees
- moved R13 227.6 mm to (117.7, 60.0), turned to 270 degrees
- moved C14 227.2 mm to (119.7, 57.9), turned to 90 degrees
- moved R38 226.3 mm to (35.7, 75.5), turned to 270 degrees
- moved R33 224.0 mm to (8.91, 62.2), turned to 0 degrees
- moved R37 223.2 mm to (42.3, 82.3)
- moved R34 222.0 mm to (8.90, 63.9), turned to 180 degrees
- moved R36 221.6 mm to (40.7, 82.3)
- moved C13 219.9 mm to (111.2, 63.4)
- moved R35 219.0 mm to (34.1, 75.5)
- moved C39 218.6 mm to (23.0, 92.6), turned to 180 degrees
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Connections:
- removed net N$94: C38.P$2, C39.P$1, E1.ANT
- new net !DSP_BL_HL: J2.7, Q7.P$3, R42.P$1
- new net !DSP_LE_HL: J2.6, Q6.P$3, R41.P$1
- new net BR2_DSP_CLK_HL: J3.5, U5.28, U6.28
- new net BRD2_!DSP_BL_HL: J3.7, U5.33, U6.33
- new net BRD2_!DSP_LE_HL: J3.6, U5.31, U6.31
- new net BRD2_12V: C16.P$1, C17.P$1, J3.3, U5.27, U5.30, U6.27, U6.30
- new net BRD2_GND2: C16.P$2, C17.P$2, J3.8, U5.29, U6.29
- new net BRD2_SDP_SDI_HL: J3.4, U5.32
- new net BRD2_VOUT: J3.1, R10.2, R11.2, R12.2, R17.2, R18.2, R9.2
- new net DSP_CLK_HL: J2.5, Q5.P$3, R40.P$1
- new net LED_GND: C41.P$2, C42.P$2, C43.P$2, C44.P$2, D2.2, D3.2, D4.2, D5.2, J5.2
- new net LED_VCC: C41.P$1, C42.P$1, C43.P$1, C44.P$1, D2.5, D3.5, D4.5, D5.5, J5.3
- new net N$21: Q4.P$1, R19.P$2
- new net N$22: Q5.P$1, R20.P$2
- new net N$24: Q7.P$1, R22.P$2
- new net N$25: Q6.P$1, R21.P$2
- new net N$26: D2.3, J5.1
- new net N$27: D2.4, J5.4
- new net N$28: C39.P$1, E1.ANT, L2.1
- new net N$29: J4.4, U11.4
- new net N$30: J4.1, U10.4
- new net N$31: D9.P$3, R43.P$2
- new net N$32: R44.P$2, R6.3, U3.2
- new net NL1: NL1.2, U6.11
- new net NL2: NL2.2, U6.12
- new net NT3-0: NT3.0, U6.1
- new net NT3-1: NT3.1, U6.2
- new net NT3-2: NT3.2, U6.3
- new net NT3-3: NT3.3, U6.4
- new net NT3-4: NT3.4, U6.5
- new net NT3-5: NT3.5, U6.6
- new net NT3-6: NT3.6, U6.7
- new net NT3-7: NT3.7, U6.8
- new net NT3-8: NT3.8, U6.9
- new net NT3-9: NT3.9, U6.10
- new net NT4-0: NT4.0, U6.35
- new net NT4-1: NT4.1, U6.36
- new net NT4-2: NT4.2, U6.37
- new net NT4-3: NT4.3, U6.38
- new net NT4-4: NT4.4, U6.39
- new net NT4-5: NT4.5, U6.40
- new net NT4-6: NT4.6, U6.41
- new net NT4-7: NT4.7, U6.42
- new net NT4-8: NT4.8, U6.43
- new net NT4-9: NT4.9, U6.44
- new net SDP_SDI_HL: J2.4, Q4.P$3, R39.P$1
- net !DSP_BL: now also R22.P$1
- net !DSP_LE: now also R21.P$1
- net 12V: now also J2.3, R39.P$2, R40.P$2, R41.P$2, R42.P$2; no longer C16.P$1, C17.P$1, U5.27, U5.30, U6.27, U6.30
- net 3.3V: now also D9.P$1, U7.3; no longer U7.2
- net 5V: now also C45.1, J4.3, U10.5, U11.5, U7.1, U9.4, U9.6; no longer D2.5, D3.5, D4.5, D5.5, U$1.4, U$1.6, U7.3
- net CHIP_PU: now also SW1.3; no longer SW1.LB, SW1.RB
- net DSP_BL_CLK: now also U11.2; no longer D2.4
- net DSP_BL_SDI: now also U10.2; no longer D2.3
- net DSP_CLK: now also R20.P$1
- net DSP_SDI: now also R19.P$1
- net GND: now also C38.P$2, C45.2, E1.GND2, J2.8, J4.2, Q4.P$2, Q5.P$2, Q6.P$2, Q7.P$2, R44.P$1, SW1.1, SW1.2, SW2.1, SW2.2, T1.1, U10.3, U11.3, U7.2, U7.4, U9.2, X2.1, X2.3; no longer C16.P$2, C17.P$2, D2.2, D3.2, D4.2, D5.2, L2.1, R6.2, SW1.LT, SW1.RT, SW2.LT, SW2.RT, U$1.2, U5.29, U6.29, U7.1, X2.2, X2.4
- net GPIO0-BOOT: now also SW2.3; no longer SW2.LB, SW2.RB
- net HFXTAL_N: now also C37.P$1, X2.4; no longer C36.P$1, X2.1
- net HFXTAL_P: now also C36.P$1, X2.2; no longer C37.P$1, X2.3
- net N$16: now also U9.1; no longer U$1.1
- net N$17: now also U9.5; no longer U$1.5
- net N$18: now also U9.3; no longer U$1.3
- net N$19: now also NL1.1; no longer NL1.2
- net N$20: now also NL2.1; no longer NL2.2
- net N$8: now also R6.2; no longer R6.1, U3.2
- net N$95: now also R43.P$1
- net VOUT: now also J2.1; no longer R10.2, R11.2, R12.2, R17.2, R18.2, R9.2
Routing:
- net 5V: track 0.00 -> 186.0 mm, vias 0 -> 4
- net BRD2_VOUT: track 0.00 -> 154.3 mm
- net 3.3V: track 0.00 -> 129.4 mm, vias 0 -> 6
- net BRD2_12V: track 0.00 -> 119.0 mm, vias 0 -> 3
- net LED_GND: track 0.00 -> 109.6 mm, vias 0 -> 7
- net LED_VCC: track 0.00 -> 108.4 mm, vias 0 -> 7
- net BR2_DSP_CLK_HL: track 0.00 -> 102.2 mm, vias 0 -> 3
- net BRD2_SDP_SDI_HL: track 0.00 -> 95.2 mm, vias 0 -> 1
- net BRD2_!DSP_LE_HL: track 0.00 -> 93.3 mm, vias 0 -> 2
- net BRD2_GND2: track 0.00 -> 92.8 mm, vias 0 -> 2
- net !HVEN: track 0.00 -> 92.7 mm, vias 0 -> 4
- net BRD2_!DSP_BL_HL: track 0.00 -> 90.4 mm, vias 0 -> 3
- net N$23: track 0.00 -> 69.7 mm, vias 0 -> 2
- net USB_DP: track 0.00 -> 66.6 mm, vias 0 -> 4
- net NT3-9: track 0.00 -> 66.1 mm
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- added copper zone on layer 1, net 5V
- added copper zone on layer 1, net GND
- added copper zone on layer 16, net GND
- added copper zone on layer 1, net N$6
Other:
- board size 130 x 50 mm -> 130 x 102 mm

Commit message: rough pcb done
Parts:
- removed LOGO2: RAFAEL_SILVA10CIRCLE, Utility > Silkscreen:RAFAEL_SILVA_10MM_CIRCLE
- removed LOGO7: RAFAEL_SILVA10MM, Utility > Silkscreen:RAFAEL_SILVA_10MM
- removed LOGO9: OSHW-LOGOL, Utility > Silkscreen:OSHW-LOGO-L
- added LOGO13: HV_WARNING, Silkscreen:HV_WARNING
- added U$1, U$2, U$3: (no value), Utility > Silkscreen:RAFAEL_SILVA_10MM_ALT
- LOGO1: value DESIGNEDINPT -> HV_WARNING; device Utility > Silkscreen:DESIGNEDINPT -> Silkscreen:HV_WARNING
- LOGO5: value RADIO-10MM -> HV_WARNING; device Silkscreen:RADIO_10MM -> Silkscreen:HV_WARNING
- moved LOGO4 76.1 mm to (41.1, 44.7)
- moved LOGO5 59.2 mm to (46.2, 44.7), flipped to the bottom
- moved LOGO1 48.6 mm to (88.9, 44.7), flipped to the bottom
- moved LOGO6 6.78 mm to (115.2, 96.0)
- moved LOGO3 4.48 mm to (18.3, 7.30)
Routing:
- net N$6: track 0.00 -> 48.2 mm
- removed copper zone on layer 1, net N$6
Other:
- board text added: "Designed in Portugal"
- board text added: "ESP32"
- board text added: "HIGH VOLTAGE DO NOT TOUCH"
- board text added: "github/gimbas"
Changed lines of the file:
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@@
 <layer number="39" name="tKeepout" color="4" fill="11" visible="no" active="yes"/>
 <layer number="40" name="bKeepout" color="1" fill="11" visible="no" active="yes"/>
-<layer number="41" name="tRestrict" color="4" fill="10" visible="no" active="yes"/>
+<layer number="41" name="tRestrict" color="4" fill="10" visible="yes" active="yes"/>
 <layer number="42" name="bRestrict" color="1" fill="10" visible="no" active="yes"/>
 <layer number="43" name="vRestrict" color="2" fill="10" visible="no" active="yes"/>
@@
 <rectangle x1="-1" y1="94.3" x2="41.9" y2="105.1" layer="41"/>
 <rectangle x1="-1" y1="94.3" x2="41.9" y2="105.1" layer="42"/>
+<text x="47.6" y="46" size="1.778" layer="21">HIGH VOLTAGE DO NOT TOUCH</text>
+<text x="7.7" y="1.9" size="1.5" layer="21" ratio="15">Designed in Portugal</text>
+<text x="56.9" y="1.4" size="1.5" layer="21" ratio="15">github/gimbas</text>
+<text x="96.6" y="95.6" size="1.778" layer="21">HIGH VOLTAGE
+DO NOT TOUCH</text>
+<text x="14.4" y="68.9" size="1.5" layer="21" ratio="15">ESP32</text>
+<text x="57.7" y="85.7" size="1.5" layer="21" ratio="15">github/gimbas</text>
+<text x="82.4" y="46" size="1.778" layer="22" rot="MR0">HIGH VOLTAGE DO NOT TOUCH</text>
+<text x="70.3" y="72.1" size="1.5" layer="22" ratio="15" rot="MR0">github/gimbas</text>
+<rectangle x1="98.3" y1="62.2" x2="105.2" y2="69.2" layer="1"/>
 </plain>
 <attributes>
@@
 <attribute name="NAME" x="47.3383" y="63.5225" size="0.8" layer="25" font="vector" ratio="15" rot="R270" align="center"/>
 </element>
-<element name="LOGO1" library="Utility &gt; Silkscreen" package="DESIGNEDINPT" value="DESIGNEDINPT" x="110.6" y="1.2" smashed="yes"/>
-<element name="LOGO2" library="Utility &gt; Silkscreen" package="RAFAEL_SILVA_10MM_CIRCLE" value="RAFAEL_SILVA10CIRCLE" x="57.2" y="85.7" smashed="yes"/>
-<element name="LOGO3" library="Utility &gt; Silkscreen" package="OSHW-LOGO-L" value="OSHW-LOGOL" x="14.2" y="9.1" smashed="yes"/>
-<element name="LOGO4" library="Silkscreen" package="HV_WARNING" value="HV_WARNING" x="116.9" y="38.4" smashed="yes"/>
-<element name="LOGO5" library="Silkscreen" package="RADIO_10MM" value="RADIO-10MM" x="1.1" y="83.1" smashed="yes"/>
-<element name="LOGO6" library="Silkscreen" package="HV_WARNING" value="HV_WARNING" x="112.7" y="89.7" smashed="yes"/>
-<element name="LOGO7" library="Utility &gt; Silkscreen" package="RAFAEL_SILVA_10MM" value="RAFAEL_SILVA10MM" x="56.3" y="4.6" smashed="yes"/>
+<element name="LOGO3" library="Utility &gt; Silkscreen" package="OSHW-LOGO-L" value="OSHW-LOGOL" x="18.3" y="7.3" smashed="yes"/>
+<element name="LOGO6" library="Silkscreen" package="HV_WARNING" value="HV_WARNING" x="115.2" y="96" smashed="yes"/>
 <element name="LOGO8" library="Utility &gt; Silkscreen" package="DESIGNEDINPT" value="DESIGNEDINPT" x="83.3" y="54.3" smashed="yes"/>
-<element name="LOGO9" library="Utility &gt; Silkscreen" package="OSHW-LOGO-L" value="OSHW-LOGOL" x="48.8" y="96.7" smashed="yes"/>
+<element name="U$1" library="Utility &gt; Silkscreen" package="RAFAEL_SILVA_10MM_ALT" value="" x="56.2" y="4" smashed="yes"/>
+<element name="LOGO4" library="Silkscreen" package="HV_WARNING" value="HV_WARNING" x="41.1" y="44.7" smashed="yes"/>
+<element name="LOGO13" library="Silkscreen" package="HV_WARNING" value="HV_WARNING" x="83.8" y="44.7" smashed="yes"/>
+<element name="U$2" library="Utility &gt; Silkscreen" package="RAFAEL_SILVA_10MM_ALT" value="" x="57" y="88.3" smashed="yes"/>
+<element name="LOGO1" library="Silkscreen" package="HV_WARNING" value="HV_WARNING" x="88.9" y="44.7" smashed="yes" rot="MR0"/>
+<element name="LOGO5" library="Silkscreen" package="HV_WARNING" value="HV_WARNING" x="46.2" y="44.7" smashed="yes" rot="MR0"/>
+<element name="U$3" library="Utility &gt; Silkscreen" package="RAFAEL_SILVA_10MM_ALT" value="" x="71" y="74.7" smashed="yes" rot="MR0"/>
 </elements>
 <signals>
@@
 <wire x1="123.535534375" y1="92.564465625" x2="125" y2="89.02893125" width="0.75" layer="1" curve="-45"/>
 <wire x1="125" y1="89.02893125" x2="125" y2="85.89" width="0.75" layer="1"/>
-<wire x1="93.375" y1="99.665" x2="92.72" y2="99.01" width="0.75" layer="1"/>
-<wire x1="92.72" y1="99.01" x2="88.75" y2="99.01" width="0.75" layer="1"/>
+<wire x1="93.375" y1="99.665" x2="91.675" y2="99.665" width="0.75" layer="1"/>
+<wire x1="91.675" y1="99.665" x2="91.02" y2="99.01" width="0.75" layer="1"/>
+<wire x1="91.02" y1="99.01" x2="88.75" y2="99.01" width="0.75" layer="1"/>
 <wire x1="88.75" y1="99.01" x2="85.1" y2="99.01" width="0.75" layer="1"/>
 <wire x1="85.1" y1="99.01" x2="85.05" y2="99.06" width="0.75" layer="1"/>
@@
 <contactref element="T1" pad="4"/>
 <contactref element="T1" pad="3"/>
-<polygon width="0.5" layer="1" rank="2">
-<vertex x="97.5" y="73.3"/>
-<vertex x="97.5" y="68.7"/>
-<vertex x="98.4" y="67.8"/>
-<vertex x="98.4" y="62.2"/>
-<vertex x="105.3" y="62.2"/>
-<vertex x="106.5" y="63.4"/>
-<vertex x="106.5" y="73.3"/>
-</polygon>
-<wire x1="103.33" y1="71.8" x2="105.83" y2="71.8" width="0" layer="19" extent="1-1"/>
-<wire x1="100.83" y1="71.8" x2="103.33" y2="71.8" width="0" layer="19" extent="1-1"/>
-<wire x1="98.33" y1="71.8" x2="100.83" y2="71.8" width="0" layer="19" extent="1-1"/>
-<wire x1="102.05" y1="64.955" x2="100.83" y2="71.8" width="0" layer="19" extent="1-1"/>
+<wire x1="98.33" y1="71.8" x2="98.33" y2="62.77" width="1" layer="1"/>
+<wire x1="98.33" y1="62.77" x2="99.3" y2="61.8" width="1" layer="1"/>
+<wire x1="99.3" y1="61.8" x2="104.2" y2="61.8" width="1" layer="1"/>
+<wire x1="105.83" y1="69.43" x2="105.83" y2="71.8" width="1" layer="1"/>
+<wire x1="104.2" y1="61.8" x2="105" y2="62.6" width="1" layer="1"/>
+<wire x1="105" y1="62.6" x2="105" y2="68.6" width="1" layer="1"/>
+<wire x1="105" y1="68.6" x2="105.83" y2="69.43" width="1" layer="1"/>
+<wire x1="105.83" y1="71.8" x2="103.33" y2="71.8" width="1" layer="1"/>
+<wire x1="103.33" y1="71.8" x2="100.83" y2="71.8" width="1" layer="1"/>
+<wire x1="100.83" y1="71.8" x2="98.33" y2="71.8" width="1" layer="1"/>
+<wire x1="102.05" y1="64.955" x2="100.83" y2="66.175" width="1" layer="1"/>
+<wire x1="100.83" y1="66.175" x2="100.83" y2="71.8" width="1" layer="1"/>
+<wire x1="102.05" y1="64.955" x2="103.33" y2="66.235" width="1" layer="1"/>
+<wire x1="103.33" y1="66.235" x2="103.33" y2="71.8" width="1" layer="1"/>
 </signal>
 <signal name="N$7">
@@
 </signals>
 <mfgpreviewcolors>
-<mfgpreviewcolor name="soldermaskcolor" color="0xC8008000"/>
+<mfgpreviewcolor name="soldermaskcolor" color="0xC8303030"/>
 <mfgpreviewcolor name="silkscreencolor" color="0xFFFEFEFE"/>
 <mfgpreviewcolor name="backgroundcolor" color="0xFF282828"/>
@@
 </drawing>
 <compatibility>
+<note version="6.3" minversion="6.2.2" severity="warning">
+Since Version 6.2.2 text objects can contain more than one line,
+which will not be processed correctly with this version.
+</note>
 <note version="8.5" severity="warning">
 Since Version 8.5, EAGLE supports locking for holes, vias, wires and polygons.

Commit message: finished board -TODO change usb connector
Parts:
- removed LOGO8: DESIGNEDINPT, Utility > Silkscreen:DESIGNEDINPT
- added LOGO2: OSHW-LOGOL, Utility > Silkscreen:OSHW-LOGO-L
- added LOGO7: HV_WARNING, Silkscreen:HV_WARNING
- moved C18 1.70 mm to (42.7, 64.7)
Routing:
- net DSP_SDI: track 1.43 -> 140.5 mm, vias 1 -> 2
- net DSP_CLK: track 1.42 -> 136.1 mm, vias 1 -> 2
- net !DSP_LE: track 1.89 -> 130.3 mm, vias 1 -> 2
- net !DSP_BL: track 1.43 -> 126.2 mm, vias 1 -> 2
- net N$6: track 48.2 -> 3.54 mm
- net GND: track 0.00 -> 37.1 mm, vias 0 -> 792
- net USB_DM: track 65.3 -> 56.8 mm
- net USB_DP: track 66.6 -> 58.2 mm, vias 4 -> 3
- net !HVEN: track 92.7 -> 86.9 mm
- net 5V: track 186.0 -> 189.7 mm, vias 4 -> 10
- net N$10: track 2.44 -> 4.09 mm
- net N$11: track 0.00 -> 1.59 mm
- net 3.3V: track 129.4 -> 130.9 mm, vias 6 -> 7
- net CHIP_PU: track 31.3 -> 32.4 mm
- net N$91: track 7.32 -> 8.08 mm
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- added copper zone on layer 1, net N$6
Other:
- board text added: "+"
- board text added: "C12"
