File: pcb/eagle_pcb/nixie_clock.brd (EAGLE design)
At the start: 130 x 102 mm, 148 parts, among them J1 USB-CVERTICAL, J2 8, J3 8, J4 4, J5 4, J6 USB-C, Q1 IRLR3110ZPBF, Q2 BC817-25, Q3 BC817-25, Q4 BC817-25, Q5 BC817-25, Q6 BC817-25, Q7 BC817-25, T1 DA2032-AL, U1 ESP32, U10 74LVC1G17, U11 74LVC1G17, U2 CP2102N, U3 LT3757, U4 DS3231, U5 HV5522, U6 HV5522, U7 MIC39100, U8 W25Q40BVSS, U9 MIC2619, X1 32.768kHz, X2 26MHz

Commit message: ready for production
Parts:
- added C46: 4n4, Passive Components > Capacitors > Multilayer Ceramic Capacitors MLCC:0603_WAVE
- added C47, C48, C49: 100n, Passive Components > Capacitors > Multilayer Ceramic Capacitors MLCC:0603_WAVE
- added R45: 1M, Passive Components > Resistors > Chip Resistors:0603_WAVE
- added R46, R47: 10k, Passive Components > Resistors > Chip Resistors:0603_WAVE
- added U12: CCS811, Sensors > Environmental Sensors > Air Quality Sensors:LGA10
- added U13: SI7021, Sensors > Humidity Sensors:DFN6
- J1: value USB-CVERTICAL -> USB-C-VVERTICAL
- J6: value USB-C -> PH-2; device Connectors > USB:USB-C -> Connectors > JST > PH:JST_PH_SMD_2
- moved J6 116.8 mm to (48.0, 98.0)
- moved C6 13.3 mm to (102.0, 97.9)
- moved C5 13.0 mm to (98.0, 97.9)
- moved R6 8.30 mm to (87.6, 91.8)
- moved R7 8.30 mm to (86.5, 96.4)
- moved R8 8.30 mm to (89.1, 97.3)
- moved R23 4.00 mm to (67.0, 54.6)
- moved R24 4.00 mm to (63.0, 54.6), turned to 0 degrees
- moved LOGO2 1.70 mm to (19.4, 60.1)
- moved U$3 1.20 mm to (72.2, 74.7)
- moved U$2 0.61 mm to (57.6, 88.4)
Connections:
- new net BTN: C47.P$1, J6.1, R46.P$1, U1.27
- new net N$33: C46.P$1, J1.S1, J1.S2, J1.S3, J1.S4, R45.P$2
- new net N$34: R47.P$1, U12.2
- new net N$35: U12.4, U12.5
- net 3.3V: now also C48.P$1, C49.P$1, R46.P$2, R47.P$2, U12.6, U13.5
- net GND: now also C46.P$2, C47.P$2, C48.P$2, C49.P$2, J1.1, J1.15, J1.16, J1.2, J6.2, R45.P$1, U12.1, U12.7, U12.PAD, U13.2; no longer J1.A1, J1.B12, J1.SHIELD0, J1.SHIELD1, J1.SHIELD2, J1.SHIELD3
- net N$74: now also J1.13, J1.14, J1.3, J1.4; no longer J1.A4, J1.A9, J1.B4, J1.B9
- net N$75: now also J1.6; no longer J1.B5
- net N$78: now also J1.11; no longer J1.A5
- net SCL: now also U12.10, U13.6
- net SDA: now also U12.9, U13.1
- net USB_DM: now also J1.10, J1.7; no longer J1.A7, J1.B7
- net USB_DP: now also J1.8, J1.9; no longer J1.A6, J1.B6
Routing:
- net BTN: track 0.00 -> 49.6 mm, vias 0 -> 2
- net 3.3V: track 130.9 -> 173.6 mm, vias 7 -> 9
- net SDA: track 34.9 -> 63.6 mm, vias 2 -> 5
- net SCL: track 33.4 -> 61.2 mm, vias 2 -> 4
- net N$74: track 11.9 -> 22.8 mm, vias 0 -> 1
- net GND: track 35.7 -> 26.7 mm, vias 786 -> 785
- net N$34: track 0.00 -> 7.37 mm
- net VOUT: track 52.7 -> 46.3 mm
- net N$33: track 0.00 -> 4.81 mm
- net N$35: track 0.00 -> 1.51 mm
- net N$78: track 4.65 -> 3.25 mm
- net N$75: track 3.33 -> 4.65 mm
- net USB_DP: track 58.0 -> 56.8 mm, vias 2 -> 1
- net USB_DM: track 55.9 -> 54.9 mm
- net N$32: track 25.3 -> 26.0 mm
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Other:
- outline, holes or cut-outs redrawn
- board text added: "#0520"
- board text added: "JLCPCBJLCPCBJLCPCB"
