File: pcb/eagle_pcb/nixie_clock.sch (EAGLE design)
At the start: 139 parts, among them J1 USB-CVERTICAL, J2 8, J3 8, J4 4, J5 4, J6 USB-C, Q1 IRLR3110ZPBF, Q2 BC817-25, Q3 BC817-25, Q4 BC817-25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

Commit message: ready for production
Parts:
- added C46: 4n4, Passive Components > Capacitors > Multilayer Ceramic Capacitors MLCC:MLCC0603
- added C47, C48, C49: 100n, Passive Components > Capacitors > Multilayer Ceramic Capacitors MLCC:MLCC0603
- added R45: 1M, Passive Components > Resistors > Chip Resistors:RESISTOR0603
- added R46, R47: 10k, Passive Components > Resistors > Chip Resistors:RESISTOR0603
- added U12: CCS811, Sensors > Environmental Sensors > Air Quality Sensors:CCS811
- added U13: SI7021, Sensors > Humidity Sensors:SI7021
- J1: value USB-CVERTICAL -> USB-C-VVERTICAL; device Connectors > USB:USB-CVERTICAL -> Connectors > USB:USB-C-VVERTICAL
- J6: value USB-C -> PH-2; device Connectors > USB:USB-C -> Connectors > JST > PH:PH-2
Connections:
- new net BTN: C47.P$1, J6.1.S, R46.P$1, U1.(HS1_DATA5)GPIO17
- new net N$33: C46.P$1, J1.SHIELD, R45.P$2
- new net N$34: R47.P$1, U12.!RESET
- new net N$35: U12.PWM, U12.SENSE
- net 3.3V: now also C48.P$1, C49.P$1, R46.P$2, R47.P$2, U12.VDD, U13.VDD
- net GND: now also C46.P$2, C47.P$2, C48.P$2, C49.P$2, J1.GND, J6.2.S, R45.P$1, U12.!WAKE, U12.ADDR, U12.GND, U13.GND; no longer J1.GND@A1,A12,B12,B1, J1.SHIELD
- net N$74: now also J1.VBUS; no longer J1.VBUS@A4,A9,B9,B4
- net N$75: now also J1.TBD2; no longer J1.CC2@B5
- net N$78: now also J1.TBD1; no longer J1.CC1@A5
- net SCL: now also U12.SCL, U13.SCL
- net SDA: now also U12.SDA, U13.SDA
- net USB_DM: now also J1.DN; no longer J1.DN@A7,B7
- net USB_DP: now also J1.DP; no longer J1.DP@A6,B6
Other:
- note added: "Air quality sensor"
- note added: "GP Button"
- note removed: "Headers"
- moved on the sheet: C18, C19, C22, C23, C24, C25, C26, C27, C28, C29, C30, C31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
